Commit message: minor

File: data/robots/atlas/atlas.urdf (robot description, URDF)
Before this commit: robot atlas, 41 links, 40 joints
Links:
- link head: geometry collision box size=0.1311 0.12 0.0591; visual box size=0.1311 0.12 0.0591
- link head_imu_link: geometry collision box size=0.01 0.01 0.01; visual box size=0.01 0.01 0.01
- link hokuyo_link: geometry collision box size=0.08 0.06 0.04238; visual box size=0.08 0.06 0.04238
- link imu_link: geometry collision box size=0.01 0.01 0.01; visual box size=0.01 0.01 0.01
- link l_clav: geometry collision mesh filename=meshes/l_clav.dae scale=1 1 1; visual mesh filename=meshes/l_clav.dae scale=1 1 1
- link l_farm: geometry collision mesh filename=meshes/l_farm.dae scale=1 1 1; visual mesh filename=meshes/l_farm.dae scale=1 1 1
- link l_foot: geometry collision mesh filename=meshes/l_foot.dae scale=1 1 1; visual mesh filename=meshes/l_foot.dae scale=1 1 1
- link l_hand: geometry collision mesh filename=meshes/l_hand.dae scale=1 1 1; visual mesh filename=meshes/l_hand.dae scale=1 1 1
- link l_larm: geometry collision mesh filename=meshes/l_larm.dae scale=1 1 1; visual mesh filename=meshes/l_larm.dae scale=1 1 1
- link l_lglut: geometry collision mesh filename=meshes/l_lglut.dae scale=1 1 1; visual mesh filename=meshes/l_lglut.dae scale=1 1 1
- link l_lleg: geometry collision mesh filename=meshes/l_lleg.dae scale=1.0 1.0 1.0; visual mesh filename=meshes/l_lleg.dae scale=1.0 1.0 1.0
- link l_scap: geometry collision mesh filename=meshes/l_scap.dae scale=1 1 1; visual mesh filename=meshes/l_scap.dae scale=1 1 1
- link l_talus: geometry collision mesh filename=meshes/l_talus.dae scale=1 1 1; visual mesh filename=meshes/l_talus.dae scale=1 1 1
- link l_uarm: geometry collision mesh filename=meshes/l_uarm.dae scale=1 1 1; visual mesh filename=meshes/l_uarm.dae scale=1 1 1
- link l_uglut: geometry collision mesh filename=meshes/l_uglut.dae scale=1 1 1; visual mesh filename=meshes/l_uglut.dae scale=1 1 1
- link l_uleg: geometry collision mesh filename=meshes/l_uleg.dae scale=1.0 1.0 1.0; visual mesh filename=meshes/l_uleg.dae scale=1.0 1.0 1.0
- link ltorso: geometry collision mesh filename=meshes/ltorso.dae scale=1 1 1; visual mesh filename=meshes/ltorso.dae scale=1 1 1
- link mtorso: geometry collision mesh filename=meshes/mtorso.dae scale=1 1 1; visual mesh filename=meshes/mtorso.dae scale=1 1 1
- link pelvis: geometry collision mesh filename=meshes/pelvis.dae scale=1.0 1.0 1.0; visual mesh filename=meshes/pelvis.dae scale=1.0 1.0 1.0
- link r_clav: geometry collision mesh filename=meshes/r_clav.dae scale=1 1 1; visual mesh filename=meshes/r_clav.dae scale=1 1 1
- link r_farm: geometry collision mesh filename=meshes/r_farm.dae scale=1 1 1; visual mesh filename=meshes/r_farm.dae scale=1 1 1
- link r_foot: geometry collision mesh filename=meshes/r_foot.dae scale=1 1 1; visual mesh filename=meshes/r_foot.dae scale=1 1 1
- link r_hand: geometry collision mesh filename=meshes/r_hand.dae scale=1 1 1; visual mesh filename=meshes/r_hand.dae scale=1 1 1
- link r_larm: geometry collision mesh filename=meshes/r_larm.dae scale=1.0 1.0 1.0; visual mesh filename=meshes/r_larm.dae scale=1.0 1.0 1.0
- link r_lglut: geometry collision mesh filename=meshes/r_lglut.dae scale=1.0 1.0 1.0; visual mesh filename=meshes/r_lglut.dae scale=1.0 1.0 1.0
- link r_lleg: geometry collision mesh filename=meshes/r_lleg.dae scale=1.0 1.0 1.0; visual mesh filename=meshes/r_lleg.dae scale=1.0 1.0 1.0
- link r_scap: geometry collision mesh filename=meshes/r_scap.dae scale=1 1 1; visual mesh filename=meshes/r_scap.dae scale=1 1 1
- link r_talus: geometry collision mesh filename=meshes/r_talus.dae scale=1 1 1; visual mesh filename=meshes/r_talus.dae scale=1 1 1
- link r_uarm: geometry collision mesh filename=meshes/r_uarm.dae scale=1.0 1.0 1.0; visual mesh filename=meshes/r_uarm.dae scale=1.0 1.0 1.0
- link r_uglut: geometry collision mesh filename=meshes/r_uglut.dae scale=1.0 1.0 1.0; visual mesh filename=meshes/r_uglut.dae scale=1.0 1.0 1.0
- link r_uleg: geometry collision mesh filename=meshes/r_uleg.dae scale=1.0 1.0 1.0; visual mesh filename=meshes/r_uleg.dae scale=1.0 1.0 1.0
- link utorso: geometry collision mesh filename=meshes/utorso.dae scale=1 1 1; visual mesh filename=meshes/utorso.dae scale=1 1 1
